File: basic_esc_carrier.kicad_pcb (KiCad board)
At the start: 2 copper layers, 17.5 x 33 mm, 15 parts, among them J1 0039301080, J10 S8B-PH-K-S, J2 0039301080, J3 Conn_02x03_Top_Bottom, J4 Conn_02x03_Top_Bottom, J5 Conn_02x03_Top_Bottom, J7 Conn_02x03_Top_Bottom, J8 Conn_02x03_Top_Bottom, J9 Conn_02x03_Top_Bottom

Commit message: started board layout, placed escs, connectors, routed some traces
Parts:
- added H1: MountingHole, MountingHole:MountingHole_3.2mm_M3, F.Cu at (238.0, 133.5)
- added H2: MountingHole, MountingHole:MountingHole_3.2mm_M3, F.Cu at (44.5, 133.5)
- added H3: MountingHole, MountingHole:MountingHole_3.2mm_M3, F.Cu at (44.5, 54.0)
- added H4: MountingHole, MountingHole:MountingHole_3.2mm_M3, F.Cu at (263.5, 80.0)
- J3, J4, J5, J7, J8, J9: footprint Connector_Molex:Molex_Mini-Fit_Jr_5569-06A1_2x03_P4.20mm_Horizontal -> Connector_Molex:Molex_Mini-Fit_Jr_5569-06A2_2x03_P4.20mm_Horizontal
- moved J9 155.6 mm to (224.5, 63.8)
- moved J8 118.5 mm to (195.4, 63.8)
- moved J2 105.4 mm to (54.3, 100.2), turned to 90 degrees
- moved J10 95.6 mm to (47.0, 111.5), turned to -90 degrees
- moved J7 81.6 mm to (166.3, 63.8)
- moved J1 74.0 mm to (54.3, 74.6), turned to 90 degrees
- moved ESC4 53.8 mm to (170.5, 124.8)
- moved ESC5 53.8 mm to (199.6, 124.8)
- moved ESC6 53.8 mm to (228.7, 124.8)
- moved ESC1 53.8 mm to (83.2, 124.8)
- moved ESC2 53.8 mm to (112.3, 124.8)
- moved ESC3 53.8 mm to (141.4, 124.8)
- moved J5 45.2 mm to (137.2, 63.8)
- moved J3 34.1 mm to (79.0, 63.8)
- moved J4 14.7 mm to (108.1, 63.8)
Connections:
- J4 pad 1: unconnected-(J4-Pin_1-Pad1) -> /ESC2_PHASE1
- J4 pad 2: unconnected-(J4-Pin_2-Pad2) -> /ESC2_PHASE2
- J4 pad 3: unconnected-(J4-Pin_3-Pad3) -> /ESC2_PHASE3
- J4 pad 4: unconnected-(J4-Pin_4-Pad4) -> /ESC2_PHASE1
- J4 pad 5: unconnected-(J4-Pin_5-Pad5) -> /ESC2_PHASE2
- J4 pad 6: unconnected-(J4-Pin_6-Pad6) -> /ESC2_PHASE3
- J5 pad 1: unconnected-(J5-Pin_1-Pad1) -> /ESC3_PHASE1
- J5 pad 2: unconnected-(J5-Pin_2-Pad2) -> /ESC3_PHASE2
- J5 pad 3: unconnected-(J5-Pin_3-Pad3) -> /ESC3_PHASE3
- J5 pad 4: unconnected-(J5-Pin_4-Pad4) -> /ESC3_PHASE1
- J5 pad 5: unconnected-(J5-Pin_5-Pad5) -> /ESC3_PHASE2
- J5 pad 6: unconnected-(J5-Pin_6-Pad6) -> /ESC3_PHASE3
- J7 pad 1: unconnected-(J7-Pin_1-Pad1) -> /ESC4_PHASE1
- J7 pad 2: unconnected-(J7-Pin_2-Pad2) -> /ESC4_PHASE2
- J7 pad 3: unconnected-(J7-Pin_3-Pad3) -> /ESC4_PHASE3
- J7 pad 4: unconnected-(J7-Pin_4-Pad4) -> /ESC4_PHASE1
- J7 pad 5: unconnected-(J7-Pin_5-Pad5) -> /ESC4_PHASE2
- J7 pad 6: unconnected-(J7-Pin_6-Pad6) -> /ESC4_PHASE3
- J8 pad 1: unconnected-(J8-Pin_1-Pad1) -> /ESC5_PHASE1
- J8 pad 2: unconnected-(J8-Pin_2-Pad2) -> /ESC5_PHASE2
- J8 pad 3: unconnected-(J8-Pin_3-Pad3) -> /ESC5_PHASE3
- J8 pad 4: unconnected-(J8-Pin_4-Pad4) -> /ESC5_PHASE1
- J8 pad 5: unconnected-(J8-Pin_5-Pad5) -> /ESC5_PHASE2
- J8 pad 6: unconnected-(J8-Pin_6-Pad6) -> /ESC5_PHASE3
- J9 pad 1: unconnected-(J9-Pin_1-Pad1) -> /ESC6_PHASE1
- J9 pad 2: unconnected-(J9-Pin_2-Pad2) -> /ESC6_PHASE2
- J9 pad 3: unconnected-(J9-Pin_3-Pad3) -> /ESC6_PHASE3
- J9 pad 4: unconnected-(J9-Pin_4-Pad4) -> /ESC6_PHASE1
- J9 pad 5: unconnected-(J9-Pin_5-Pad5) -> /ESC6_PHASE2
- J9 pad 6: unconnected-(J9-Pin_6-Pad6) -> /ESC6_PHASE3
Routing:
- net /ESC6_SIGNAL: track 0.00 -> 189.4 mm
- net /ESC5_SIGNAL: track 0.00 -> 159.5 mm
- net /ESC4_SIGNAL: track 0.00 -> 129.5 mm
- net /ESC3_SIGNAL: track 0.00 -> 99.6 mm
- net /ESC2_SIGNAL: track 0.00 -> 69.7 mm
- net /ESC1_SIGNAL: track 0.00 -> 43.0 mm
- net /ESC5_PHASE3: track 0.00 -> 12.7 mm
- net /ESC4_PHASE3: track 0.00 -> 12.7 mm
- net /ESC3_PHASE3: track 0.00 -> 12.7 mm
- net /ESC1_PHASE3: track 0.00 -> 12.7 mm
- net /ESC2_PHASE3: track 0.00 -> 12.7 mm
- net /ESC6_PHASE3: track 0.00 -> 12.7 mm
- net /ESC6_PHASE1: track 0.00 -> 12.7 mm
- net /ESC5_PHASE1: track 0.00 -> 12.7 mm
- net /ESC2_PHASE1: track 0.00 -> 12.7 mm
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- added copper zone on B.Cu, net GND
- added copper zone on F.Cu, net VBAT
Other:
- board size 17.5 x 33 mm -> 203.2 x 88.9 mm
